File: KiCad/level_converter.kicad_sch (KiCad schematic)
At the start: 3 parts, among them Q2 BSS138

Commit message: Final review before PCB manufacturing
Parts:
- renumbered Q2 to Q1
Changed lines of the file:
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@@
   (symbol (lib_id "power:+5V") (at 113.03 53.34 0) (unit 1)
     (in_bom yes) (on_board yes)
-    (property "Reference" "#PWR021" (id 0) (at 113.03 57.15 0)
+    (property "Reference" "#PWR020" (id 0) (at 113.03 57.15 0)
       (effects (font (size 1.27 1.27)) hide)
     )
@@
   (symbol (lib_id "Transistor_FET:BSS138") (at 101.6 67.31 270) (unit 1)
     (in_bom yes) (on_board yes)
-    (property "Reference" "Q2" (id 0) (at 107.95 72.39 90))
+    (property "Reference" "Q1" (id 0) (at 107.95 72.39 90))
     (property "Value" "BSS138" (id 1) (at 93.98 72.39 90))
     (property "Footprint" "Package_TO_SOT_SMD:SOT-23" (id 2) (at 99.695 72.39 0)
@@
   (symbol (lib_id "power:+3.3V") (at 101.6 53.34 0) (unit 1)
     (in_bom yes) (on_board yes)
-    (property "Reference" "#PWR020" (id 0) (at 101.6 57.15 0)
+    (property "Reference" "#PWR019" (id 0) (at 101.6 57.15 0)
       (effects (font (size 1.27 1.27)) hide)
     )
