File: KiCad/sharp-ce140f-emul_v1.kicad_sch (KiCad schematic)
At the start: 28 parts, among them J2 Micro_SD_Card_Det, J3 Conn_01x15, J4 Conn_01x15, J5 Conn_01x01, J6 Conn_01x01, J7 Conn_01x01, J8 Sharp PC 11-pin, J9 Conn_01x01, U2 NUCLEO-L053R8, U3 NUCLEO-L432KC

Commit message: PCB review
Parts:
- D2, D3, D4, D5: footprint Diode_SMD:D_0805_2012Metric_Pad1.15x1.40mm_HandSolder -> Diode_SMD:D_SOD-323_HandSoldering
Changed lines of the file:
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@@
     (effects (font (size 1.27 1.27)) (justify left bottom))
   )
-  (label "CN4_7" (at 149.86 105.41 0)
+  (label "CN4_7" (at 134.62 105.41 0)
     (effects (font (size 1.27 1.27)) (justify left bottom))
   )
@@
       (effects (font (size 1.27 1.27)) (justify left))
     )
-    (property "Footprint" "Diode_SMD:D_0805_2012Metric_Pad1.15x1.40mm_HandSolder" (id 2) (at 231.14 78.74 0)
+    (property "Footprint" "Diode_SMD:D_SOD-323_HandSoldering" (id 2) (at 231.14 78.74 0)
       (effects (font (size 1.27 1.27)) hide)
     )
@@
       (effects (font (size 1.27 1.27)) (justify left))
     )
-    (property "Footprint" "Diode_SMD:D_0805_2012Metric_Pad1.15x1.40mm_HandSolder" (id 2) (at 231.14 100.33 0)
+    (property "Footprint" "Diode_SMD:D_SOD-323_HandSoldering" (id 2) (at 231.14 100.33 0)
       (effects (font (size 1.27 1.27)) hide)
     )
@@
       (effects (font (size 1.27 1.27)) (justify left))
     )
-    (property "Footprint" "Diode_SMD:D_0805_2012Metric_Pad1.15x1.40mm_HandSolder" (id 2) (at 231.14 88.9 0)
+    (property "Footprint" "Diode_SMD:D_SOD-323_HandSoldering" (id 2) (at 231.14 88.9 0)
       (effects (font (size 1.27 1.27)) hide)
     )
@@
       (effects (font (size 1.27 1.27)) (justify left))
     )
-    (property "Footprint" "Diode_SMD:D_0805_2012Metric_Pad1.15x1.40mm_HandSolder" (id 2) (at 231.14 68.58 0)
+    (property "Footprint" "Diode_SMD:D_SOD-323_HandSoldering" (id 2) (at 231.14 68.58 0)
       (effects (font (size 1.27 1.27)) hide)
     )
@@
     )
     (path "/fdb96423-19c0-483a-89a4-bb44582e187d"
-      (reference "D2") (unit 1) (value "1N4148") (footprint "Diode_SMD:D_0805_2012Metric_Pad1.15x1.40mm_HandSolder")
+      (reference "D2") (unit 1) (value "1N4148") (footprint "Diode_SMD:D_SOD-323_HandSoldering")
     )
     (path "/0835fd48-14bd-4511-a471-b9bb9f0d0b70"
-      (reference "D3") (unit 1) (value "1N4148") (footprint "Diode_SMD:D_0805_2012Metric_Pad1.15x1.40mm_HandSolder")
+      (reference "D3") (unit 1) (value "1N4148") (footprint "Diode_SMD:D_SOD-323_HandSoldering")
     )
     (path "/b16fd4c8-0cd7-45e4-bb95-3013119f0754"
-      (reference "D4") (unit 1) (value "1N4148") (footprint "Diode_SMD:D_0805_2012Metric_Pad1.15x1.40mm_HandSolder")
+      (reference "D4") (unit 1) (value "1N4148") (footprint "Diode_SMD:D_SOD-323_HandSoldering")
     )
     (path "/3a193148-e006-43e4-9cd0-5ea62451216c"
-      (reference "D5") (unit 1) (value "1N4148") (footprint "Diode_SMD:D_0805_2012Metric_Pad1.15x1.40mm_HandSolder")
+      (reference "D5") (unit 1) (value "1N4148") (footprint "Diode_SMD:D_SOD-323_HandSoldering")
     )
     (path "/d836a490-6890-4e2b-99b2-610cda381e75"

Commit message: some footprint review and BOM exported (csv)
Parts:
- BTN1: footprint Button_Switch_THT:SW_PUSH_6mm -> Button_Switch_SMD:SW_Push_1P1T_NO_6x6mm_H9.5mm
Changed lines of the file:
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@@
     (property "Reference" "BTN1" (id 0) (at 160.02 76.2 0))
     (property "Value" "User_button" (id 1) (at 160.02 78.74 0))
-    (property "Footprint" "Button_Switch_THT:SW_PUSH_6mm" (id 2) (at 160.02 78.74 0)
+    (property "Footprint" "Button_Switch_SMD:SW_Push_1P1T_NO_6x6mm_H9.5mm" (id 2) (at 160.02 78.74 0)
       (effects (font (size 1.27 1.27)) hide)
     )
@@
     )
     (path "/b95a3306-bcc2-49a6-b437-3786461cf2e6"
-      (reference "BTN1") (unit 1) (value "User_button") (footprint "Button_Switch_THT:SW_PUSH_6mm")
+      (reference "BTN1") (unit 1) (value "User_button") (footprint "Button_Switch_SMD:SW_Push_1P1T_NO_6x6mm_H9.5mm")
     )
     (path "/31308ac8-906a-485c-b104-416b7e839401"

Commit message: Final review before PCB manufacturing
Parts:
- added R4: 47k, Resistor_SMD:R_0603_1608Metric_Pad0.98x0.95mm_HandSolder, symbol Device:R_Small
- renumbered C2 to C1, C3 to C2, D2 to D1, D3 to D2, D4 to D3, D5 to D4, J9 to J1, BTN1 to PB1, R2 to R1, R3 to R2, R4 to R3, U2 to U1, U3 to U2
Connections:
- net sd_sck is gone; now on net CN4_8: J2.5 (CLK), R2.2
- net +3V3: now also R4.1
- net CN3_14: now also J2.2 (DAT3/CD), R4.2; no longer J2.3 (CMD)
- net CN4_6: now also J2.3 (CMD), R3.2, U1.CN9_5 (D4)
- net CN4_7: now also J2.7 (DAT0), R1.2, U1.CN9_6 (D5); no longer J2.2 (DAT3/CD), R3.2, U1.CN9_5 (D4)
- net CN4_8: no longer J2.7 (DAT0), R1.2, U1.CN9_6 (D5)
Other:
- note added: "(*) Cut jumpers to use SPI on these lines By default the PA_5 (A4) and PA_6 (A5) pins can only be used as Input floating (ADC function). See L432KC Manual"
- note removed: "(*) Cut jumpers to use SPI on these lines See L432KC Manual"
- moved on the sheet: C1, C2, J1, R2, R3, R5
