File: level_conv_sim/level_conv.kicad_sch (KiCad schematic)
At the start: 32 parts, among them Q1 BSS138, Q2 DTA144E, Q3 DTC144E, Q4 BSS138

Commit message: Fixed simulation design
Parts:
- removed D1: CUHS20S30, symbol pspice:DIODE
- removed MN3, MN9: cmosn, symbol pspice:MNMOS
- removed MP3, MP9: cmosp, symbol pspice:MPMOS
- removed R5, R9: 1M, symbol pspice:R
- Rpu: value 10k -> 3k; Spice_Model 10k -> 3k
Connections:
- net VCC is gone; now on net +BATT: MP1.3 (S), MP1.4 (B)
- net 0: no longer MN1.3 (S), MN1.4 (B), Q3.3 (E)
- net sharp_in_value: now also MN1.1 (D), MP1.1 (D)
- net +BATT: now reaches C1.2, Vbatt1.1 (E1)
- net -BATT: now reaches R4.1, Vbatt1.2 (E2)
- net -BATT: now also MN1.3 (S), MN1.4 (B), Q3.3 (E)
Other:
- note added: "NGSPICE simulation:"
- note removed: "Schottky"
- moved on the sheet: C3, D3, MN1, MN2, MP1, MP2, Q2, Q3, S2A, V_pulse1, V_pulse2, Vcc1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
